File: Hardware/Design/14226.brd (EAGLE design)
At the start: 60.3 x 53.3 mm, 77 parts, among them J1 RJ45J, J2 PBC10SAAN, J4 RJ45J, J5 PBC10SAAN, J6 PBC10SAAN, J7 PBC08SAAN, J8 PPPC032LFBN, Q1 K38, Q2 K38, Q3 K38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

Commit message: Hardware: ^5 review
Parts:
- added TP1, TP2, TP3: TPPAD1-08, J-TP:P1-08
Connections:
- new net SHUTDWN: TP1.TP, U7.12
- net DTR_RXD: now also TP3.TP; no longer U7.12
- net DTR_TXD: now also TP2.TP
Routing:
- net SHUTDWN: track 0.00 -> 10.3 mm, vias 0 -> 1
- net MOSI: track 43.7 -> 48.6 mm
- net DTR_RXD: track 90.4 -> 87.8 mm, vias 5 -> 4
- net HOST_TX: track 57.0 -> 55.1 mm
- net !SS!: track 30.0 -> 31.6 mm
- net SCK: track 51.1 -> 52.5 mm
- net 0V: vias 50 -> 51
Other:
- board text added: "14226^5"
- board text added: "DTR RXD"
- board text added: "DTR TXD"
- board text added: "ICP1"
- board text added: "RPUBUS.ORG"
- board text removed: "14226^4"
- board text removed: "EPCCS.ORG"

Commit message: Hardware: ^5 more review
Parts:
- removed C13: 15pF, C-C:C0603(1608)
- removed D3: 0805RD, D-LED:C0805(2012)
- removed R30: 10k, R-C:C0805(2012)
- removed R31: 1.5k, R-C:C0805(2012)
- C10: value 0.1uF -> .1uF
- C11: value .1uF -> 15pF
- C3: value 0.1uF -> 470pF
- C4: value 470pF -> 10uF; device C-C:C0603(1608) -> C-T:3216
- C5: value 10uF -> .1uF; device C-T:3216 -> C-C:C0603(1608)
- C9: value .1uF -> 0.1uF
- D1: value SQ4 -> T4; device D-SBR:SMA -> D-GP:SOD123
- D2: value T4 -> 0805RD; device D-GP:SOD123 -> D-LED:C0805(2012)
- R14: value 200k -> OPEN
- R15: value 10k -> 3.01k
- R16: value OPEN -> 10k
- R17: value 3.01k -> 10k
- R18: value 10k -> 100
- R19: value 10k -> 10K
- R20: value 100 -> 182
- R21, R24: value 10K -> 3.01k
- R22: value 182 -> 10K
- R25, R26: value 3.01k -> 182
- R27: value 182 -> 100k
- R28: value 182 -> 10k
- R29: value 100k -> 1.5k
- Y1: value 14.7456MHz -> 12MHz
- moved R29 54.2 mm to (56.5, 33.0), turned to 180 degrees
- moved D1 48.2 mm to (55.6, 38.7), turned to 180 degrees
- moved R21 40.2 mm to (32.6, 8.38), turned to 90 degrees
- moved R23 40.1 mm to (42.0, 47.4), turned to 270 degrees
- moved R19 39.3 mm to (47.8, 45.6)
- moved R20 36.7 mm to (50.5, 47.9)
- moved R26 33.7 mm to (8.51, 46.6), turned to 0 degrees
- moved R25 33.4 mm to (8.64, 48.6), turned to 0 degrees
- moved C9 31.9 mm to (7.62, 18.3), turned to 180 degrees
- moved R15 30.9 mm to (40.1, 20.8)
- moved C7 30.4 mm to (25.9, 36.2), turned to 0 degrees
- moved R27 28.5 mm to (3.81, 20.6)
- moved R18 28.3 mm to (32.9, 15.7), turned to 270 degrees
- moved C10 28.0 mm to (27.4, 38.1), turned to 0 degrees
- moved R28 26.4 mm to (7.62, 20.2), turned to 180 degrees
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Connections:
- removed net IOREF_ADC6: C10.1, R29.1, R30.1, U7.19
- removed net N$1: D1.A, J3.3
- removed net VIN_ADC7: C3.1, R14.2, R15.1, U7.22
- new net 5V_ADC6: C9.1, R27.1, R28.1, U7.19
- net +3V3: now also C4.+, C5.1, D1.C, R16.2, R17.2, R22.2, R23.1, R24.1, R29.1; no longer C5.+, C9.1, D2.C, R18.2, R19.2, R24.2, R25.1, R26.1, R31.1
- net +5V: now also J3.3, R27.2; no longer D1.K, R14.1
- net +RX: now also R14.1; no longer R16.1
- net -RX: now also R14.2; no longer R16.2
- net 0V: now also C4.-, C5.2, R28.2; no longer C13.2, C4.2, C5.-, R17.2, R30.2
- net HOST_TX: now also R16.1; no longer R20.1
- net IOREF: now also R19.1; no longer R21.1, R29.2
- net LED_BUILTIN: now also D2.K; no longer D3.K
- net MGR_!RESET: now also D1.A, R22.1; no longer D2.A, R24.1
- net N$10: now also R19.2, R20.2; no longer R21.2, R22.2
- net N$11: now also R21.2; no longer R23.2
- net N$24: now also C3.1; no longer C4.1
- net N$25: now also R18.2; no longer R20.2
- net N$29: now also D2.A, R29.2; no longer D3.A, R31.2
- net RPU_AREF: now also C10.1; no longer C11.1
- net RX: now also R20.1; no longer R22.1
- net RX_!RE: now also R15.1; no longer R17.1
- net RX_DE: now also R21.1; no longer R23.1
- net RX_RPU: now also R17.1; no longer R19.1
- net SCL: now also R26.2; no longer R28.2
- net SCL0: now also R24.2, R26.1; no longer R26.2, R28.1
- net SDA: now also R25.2; no longer R27.2
- net SDA0: now also R23.2, R25.1; no longer R25.2, R27.1
- net XTAL1: now also C11.1; no longer C12.1
- net XTAL2: now also C12.1; no longer C13.1
Routing:
- net IOREF_ADC6: track 37.2 -> 0.00 mm, vias 4 -> 0
- net 5V_ADC6: track 0.00 -> 37.2 mm, vias 0 -> 4
- net VIN_ADC7: track 34.8 -> 0.00 mm, vias 2 -> 0
- net IOREF: track 128.0 -> 100.3 mm, vias 4 -> 3
- net +5V: track 50.3 -> 70.6 mm
- net N$1: track 2.75 -> 0.00 mm
- net 0V: vias 51 -> 52
Other:
- board text added: "+5V"
- board text removed: "HOST_5V"
