File: Hardware/Design/14226.sch (EAGLE design)
At the start: 77 parts, among them J1 RJ45J, J2 PBC10SAAN, J4 RJ45J, J5 PBC10SAAN, J6 PBC10SAAN, J7 PBC08SAAN, J8 PPPC032LFBN, Q1 K38, Q2 K38, Q3 K38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

Commit message: Hardware: ^5 review
Parts:
- added TP1, TP2, TP3: TPPAD1-08, J-TP:TPPAD1-08
Connections:
- new net SHUTDWN: TP1.TP, U7.(ICP1)PB0
- net DTR_RXD: now also TP3.TP; no longer U7.(ICP1)PB0
- net DTR_TXD: now also TP2.TP
Other:
- note added: "1/14/17"
- note added: "BUS MANAGER NEEDS TO PULL UP DTR_DE TO ALLOW DTR_TXD TO DRIVE DTR PAIR"
- note added: "BUS MANAGER NEEDS TO PULL UP RX_DE TO ALLOW HOST_TX TO DRIVE RX PAIR"
- note added: "BUS MANAGER NEEDS TO PULL UP TX_DE TO ALLOW HOST_RX TO DRIVE TX PAIR"
- note added: "ICP1 TO TP"
- note added: "^5"
- note removed: "BUS MANAGER MUST PULL UP TO ALLOW HOST TO DRIVE RX PAIR"
- note removed: "BUS MANAGER MUST PULL UP TO ALLOW MCU NODE BOARD TO DRIVE TX PAIR"
- note removed: "BUS MANAGER NEEDS TO DRIVE DTR_DE BUT A HIGH DTR_TXD OVERIDES"
Changed lines of the file:
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@@
 <part name="R18" library="R-C" deviceset="R" device="0805" value="10k"/>
 <part name="GND1" library="Plane" deviceset="0V" device=""/>
+<part name="TP1" library="J-TP" deviceset="TP" device="PAD1-08"/>
+<part name="TP2" library="J-TP" deviceset="TP" device="PAD1-08"/>
+<part name="TP3" library="J-TP" deviceset="TP" device="PAD1-08"/>
 </parts>
 <sheets>
@@
 <text x="356.87" y="26.416" size="2.54" layer="98">SHIELD FOR RPU BUS
 RS-422 + RS-485 NODE</text>
-<text x="350.012" y="41.656" size="2.54" layer="98">RON S</text>
-<text x="335.788" y="41.656" size="2.1844" layer="98">9/29/16</text>
+<text x="350.012" y="44.196" size="2.54" layer="98">RON S</text>
+<text x="335.788" y="44.196" size="2.1844" layer="98">1/14/17</text>
 <text x="365.76" y="20.32" size="2.54" layer="98">RPUADPT</text>
 <text x="363.982" y="188.468" size="1.27" layer="98">IO13</text>
@@
 <text x="298.958" y="234.95" size="1.27" layer="98">10k PULLUP CAN BE USED
 WITHOUT MCU BOARD</text>
-<text x="306.578" y="214.63" size="1.27" layer="98">BUS MANAGER MUST
-PULL UP TO ALLOW
-MCU NODE BOARD TO
-DRIVE TX PAIR </text>
+<text x="296.418" y="214.63" size="1.27" layer="98">BUS MANAGER NEEDS TO
+PULL UP TX_DE TO ALLOW
+HOST_RX TO DRIVE TX PAIR </text>
 <text x="307.34" y="190.246" size="1.27" layer="98">BUS MANAGER NEEDS
-TO DRIVE DTR_DE
-BUT A HIGH DTR_TXD
-OVERIDES</text>
+TO PULL UP DTR_DE TO
+ALLOW DTR_TXD
+TO DRIVE DTR PAIR</text>
 <text x="205.74" y="45.72" size="1.778" layer="98">32TQFPpin
     ATTMEGA328P reg-bit
@@
 <text x="112.776" y="92.964" size="1.778" layer="98">*</text>
 <text x="115.062" y="98.552" size="1.778" layer="98">*</text>
-<text x="311.658" y="151.13" size="1.27" layer="98">BUS MANAGER MUST
-PULL UP TO ALLOW
-HOST TO DRIVE
-RX PAIR </text>
+<text x="311.658" y="151.13" size="1.27" layer="98">BUS MANAGER NEEDS TO
+PULL UP RX_DE TO ALLOW
+HOST_TX TO DRIVE RX PAIR </text>
 <text x="240.538" y="209.55" size="1.27" layer="98">BUS MANAGER MAY
 PULL UP TX_!RE! TO
@@
 PWR FROM +5V, RM SMPS</text>
 <text x="320.548" y="26.67" size="1.778" layer="98">9/29/16</text>
+<text x="282.702" y="32.004" size="2.54" layer="98">^5</text>
+<text x="290.068" y="30.988" size="1.6764" layer="98">ICP1 TO TP</text>
+<text x="320.548" y="31.75" size="1.778" layer="98">1/14/17</text>
 </plain>
 <instances>
@@
 <instance part="R18" gate="G$1" x="241.3" y="139.7" rot="R180"/>
 <instance part="GND1" gate="1" x="27.94" y="203.2"/>
+<instance part="TP1" gate="G$1" x="109.22" y="71.12"/>
+<instance part="TP2" gate="G$1" x="287.02" y="190.5"/>
+<instance part="TP3" gate="G$1" x="292.1" y="208.28"/>
 </instances>
 <busses>
@@
 <net name="TX_DE" class="0">
 <segment>
-<label x="297.18" y="218.44" size="1.27" layer="91" xref="yes"/>
+<label x="284.48" y="218.44" size="1.27" layer="91" xref="yes"/>
 <pinref part="R4" gate="G$1" pin="2"/>
-<wire x1="279.4" y1="218.44" x2="297.18" y2="218.44" width="0.1524" layer="91"/>
+<wire x1="279.4" y1="218.44" x2="284.48" y2="218.44" width="0.1524" layer="91"/>
 </segment>
 <segment>
@@
 <label x="297.18" y="205.74" size="1.27" layer="91" xref="yes"/>
 <pinref part="R13" gate="G$1" pin="2"/>
-<wire x1="287.02" y1="205.74" x2="297.18" y2="205.74" width="0.1524" layer="91"/>
+<wire x1="287.02" y1="205.74" x2="292.1" y2="205.74" width="0.1524" layer="91"/>
+<pinref part="TP3" gate="G$1" pin="TP"/>
+<wire x1="292.1" y1="205.74" x2="297.18" y2="205.74" width="0.1524" layer="91"/>
+<junction x="292.1" y="205.74"/>
 </segment>
 <segment>
@@
 <wire x1="96.52" y1="91.44" x2="96.52" y2="93.98" width="0.1524" layer="91"/>
 <wire x1="96.52" y1="93.98" x2="99.06" y2="93.98" width="0.1524" layer="91"/>
-</segment>
-<segment>
-<pinref part="U7" gate="G$1" pin="(ICP1)PB0"/>
-<wire x1="96.52" y1="68.58" x2="99.06" y2="68.58" width="0.1524" layer="91"/>
-<label x="99.06" y="68.58" size="1.27" layer="91" xref="yes"/>
 </segment>
 </net>
@@
 <wire x1="279.4" y1="182.88" x2="279.4" y2="187.96" width="0.1524" layer="91"/>
 <junction x="279.4" y="187.96"/>
-<wire x1="279.4" y1="187.96" x2="297.18" y2="187.96" width="0.1524" layer="91"/>
+<wire x1="279.4" y1="187.96" x2="287.02" y2="187.96" width="0.1524" layer="91"/>
+<pinref part="TP2" gate="G$1" pin="TP"/>
+<wire x1="287.02" y1="187.96" x2="297.18" y2="187.96" width="0.1524" layer="91"/>
+<junction x="287.02" y="187.96"/>
 </segment>
 <segment>
@@
 </segment>
 </net>
+<net name="SHUTDWN" class="0">
+<segment>
+<pinref part="U7" gate="G$1" pin="(ICP1)PB0"/>
+<wire x1="96.52" y1="68.58" x2="109.22" y2="68.58" width="0.1524" layer="91"/>
+<pinref part="TP1" gate="G$1" pin="TP"/>
+</segment>
+</net>

Commit message: Hardware: ^5 more review
Parts:
- removed C13: 15pF, C-C:CC0603A
- removed D3: 0805RD, D-LED:LEDC0805(2012)
- removed R30: 10k, R-C:R0805
- removed R31: 1.5k, R-C:R0805
- C10: value 0.1uF -> .1uF
- C11: value .1uF -> 15pF
- C3: value 0.1uF -> 470pF
- C4: value 470pF -> 10uF; device C-C:CC0603A -> C-T:CT1206
- C5: value 10uF -> .1uF; device C-T:CT1206 -> C-C:CC0603A
- C9: value .1uF -> 0.1uF
- D1: value SQ4 -> T4; device D-SBR:DSMA -> D-GP:DSOD123
- D2: value T4 -> 0805RD; device D-GP:DSOD123 -> D-LED:LEDC0805(2012)
- R14: value 200k -> OPEN
- R15: value 10k -> 3.01k
- R16: value OPEN -> 10k
- R17: value 3.01k -> 10k
- R18: value 10k -> 100
- R19: value 10k -> 10K
- R20: value 100 -> 182
- R21, R24: value 10K -> 3.01k
- R22: value 182 -> 10K
- R25, R26: value 3.01k -> 182
- R27: value 182 -> 100k
- R28: value 182 -> 10k
- R29: value 100k -> 1.5k
- Y1: value 14.7456MHz -> 12MHz
Connections:
- removed net IOREF_ADC6: C10.1, R29.1, R30.1, U7.(ICP3/!SS1!)PE2
- removed net N$1: D1.A, J3.5V
- removed net VIN_ADC7: C3.1, R14.2, R15.1, U7.(A7/T3/MOSI1)PE3
- new net 5V_ADC6: C9.1, R27.1, R28.1, U7.(ICP3/!SS1!)PE2
- net +3V3: now also C4.+, C5.1, D1.K, R16.2, R17.2, R22.2, R23.1, R24.1, R29.1; no longer C5.+, C9.1, D2.K, R18.2, R19.2, R24.2, R25.1, R26.1, R31.1
- net +5V: now also J3.5V, R27.2; no longer D1.K, R14.1
- net +RX: now also R14.1; no longer R16.1
- net -RX: now also R14.2; no longer R16.2
- net 0V: now also C4.-, C5.2, R28.2; no longer C13.2, C4.2, C5.-, R17.2, R30.2
- net HOST_TX: now also R16.1; no longer R20.1
- net IOREF: now also R19.1; no longer R21.1, R29.2
- net LED_BUILTIN: now also D2.K; no longer D3.K
- net MGR_!RESET: now also D1.A, R22.1; no longer D2.A, R24.1
- net N$10: now also R19.2, R20.2; no longer R21.2, R22.2
- net N$11: now also R21.2; no longer R23.2
- net N$24: now also C3.1; no longer C4.1
- net N$25: now also R18.2; no longer R20.2
- net N$29: now also D2.A, R29.2; no longer D3.A, R31.2
- net RPU_AREF: now also C10.1; no longer C11.1
- net RX: now also R20.1; no longer R22.1
- net RX_!RE: now also R15.1; no longer R17.1
- net RX_DE: now also R21.1; no longer R23.1
- net RX_RPU: now also R17.1; no longer R19.1
- net SCL: now also R26.2; no longer R28.2
- net SCL0: now also R24.2, R26.1; no longer R26.2, R28.1
- net SDA: now also R25.2; no longer R27.2
- net SDA0: now also R23.2, R25.1; no longer R25.2, R27.1
- net XTAL1: now also C11.1; no longer C12.1
- net XTAL2: now also C12.1; no longer C13.1
Other:
- note added: "1/24/17"
- note added: "CRYSTAL: ECS-120-20-3X-TR 12MHZ +/- 30PPM STABILITY AND TOLERANCE CRYSTAL CAPACITORS: 15PF = 5PF + (20PF*20PF)/(20PF+20PF)"
- note added: "ICP1 TO TP, ADD CRYSTAL"
- note removed: "1/14/17"
- note removed: "4.98mV/V"
- note removed: "CRYSTAL NOT USED: ECS-147.4-20-3X-TR 14.7456MHZ +/- 30PPM STABILITY AND TOLERANCE CRYSTAL CAPACITORS: 15PF = 5PF + (20PF*20PF)/(20PF+20PF)"
- note removed: "ICP1 TO TP"
- moved on the sheet: C10, C11, C12, C3, C6, C7, C8, C9, R14, R15, R16, R17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
