File: Hardware/Design/MultiDrop.sch (EAGLE design)
At the start: 13 parts

Commit message: Hardware: ^5 more review
Parts:
- removed BM1, BM3: (no value), Documentation:RPUNO
- removed PV1: PV, Documentation:PV
- added PM1: (no value), Documentation:DESKTOP
- added UART1: (no value), Documentation:UART
- U$3: value PI -> IRRIGATE7; device Documentation:PI -> Documentation:IRRIGATE7
- U$4: value BAT -> BUS_MGR; device Documentation:BAT -> Documentation:BUS_MGR
- U$5: value BUS_MGR -> IRRIGATE7; device Documentation:BUS_MGR -> Documentation:IRRIGATE7
Connections:
- removed net N$12: BM2.BAT, U$4.BAT_PWR
- removed net N$41: BM3.SHLD_5V, U$5.PWR
- new net N$13: U$1.PWR, U$3.SHLD_5V
- net +DTR: now also U$4.+DTR; no longer U$1.+DTR
- net +DTR3: now also U$1.+DTR; no longer U$5.+DTR
- net +RX: now also U$4.+RX; no longer U$1.+RX
- net +RX3: now also U$1.+RX; no longer U$5.+RX
- net +TX: now also U$4.+TX; no longer U$1.+TX
- net +TX3: now also U$1.+TX; no longer U$5.+TX
- net -DTR: now also U$4.-DTR; no longer U$1.-DTR
- net -DTR3: now also U$1.-DTR; no longer U$5.-DTR
- net -RX: now also U$4.-RX; no longer U$1.-RX
- net -RX3: now also U$1.-RX; no longer U$5.-RX
- net -TX: now also U$4.-TX; no longer U$1.-TX
- net -TX3: now also U$1.-TX; no longer U$5.-TX
- net N$1: now also U$4.BM_TX; no longer U$1.BM_TX
- net N$10: now also U$5.TX; no longer BM1.TX
- net N$11: now also U$5.RX; no longer BM1.RX
- net N$14: now also U$1.BM_TX, U$3.TX; no longer BM3.TX, U$5.BM_TX
- net N$17: now also U$5.BAT; no longer BM1.BAT
- net N$2: now also U$4.BM_RX; no longer U$1.BM_RX
- net N$21: now also U$1.BM_RX, U$3.RX; no longer BM3.RX, U$5.BM_RX
- net N$29: now also U$4.PWR, UART1.5V; no longer U$1.PWR
- net N$3: now also PM1.RX, UART1.USB; no longer BM2.SHLD_VIN, U$3.PWR
- net N$30: now also BM2.!RESET, U$4.DIO10; no longer BM2.RESET, U$1.DIO
- net N$31: now also U$3.BAT; no longer BM3.BAT
- net N$32: now also U$1.I2C, U$3.I2C; no longer BM3.I2C, U$5.I2C
- net N$33: now also U$4.I2C; no longer U$1.I2C
- net N$34: now also U$3.PV; no longer BM3.PV
- net N$36: now also U$5.PV; no longer BM1.PV
- net N$4: now also U$4.!CTS, UART1.!CTS; no longer U$1.!CTS, U$3.CTS
- net N$43: now also U$1.DIO10, U$3.!RESET; no longer BM3.RESET, U$5.DIO
- net N$44: now also U$2.DIO10, U$5.!RESET; no longer BM1.RESET, U$2.DIO
- net N$45: now also U$5.SHLD_5V; no longer BM1.SHLD_5V
- net N$48: now also U$5.I2C; no longer BM1.I2C
- net N$5: now also U$4.!RTS, UART1.!RTS; no longer U$1.!RTS, U$3.RTS
- net N$6: now also U$4.!DTR, UART1.!DTR; no longer BM2.SPI, U$3.SPI
- net N$7: now also U$4.!DSR, UART1.!DSR; no longer BM2.PV, PV1.PV_PWR
- net N$8: now also U$4.HOST_RX, UART1.RX; no longer U$1.PM_RX
- net N$9: now also U$4.HOST_TX, UART1.TX; no longer U$1.PM_TX
Other:
- note added: "RPUftdi"
- note removed: "RPU BUS"
- note removed: "RPUpi"
